File: beaglebone-can-r1.kicad_pcb (KiCad board)
At the start: 2 copper layers, 86.4 x 54.6 mm, 42 parts, among them P1 BEAGLEBONE_BLACK, P2 PINBALL-CONNECTOR, P3 PINBALL-CONNECTOR, U1 MCP2562, U2 24C256, U3 AP3513E

Commit message: A bunch of old updates
Parts:
- moved REF** 50.9 mm to (183.2, 101.0)
- moved P3 3.49 mm to (236.2, 99.7)
- moved P2 2.54 mm to (236.2, 82.9)
- turned D1 to 0 degrees
- turned D2 to 0 degrees
- turned D3 to 0 degrees
Connections:
- D1 pad 1: Net-(D1-Pad1) -> GND
- D1 pad 2: GND -> Net-(D1-Pad2)
- D2 pad 1: Net-(D2-Pad1) -> GND
- D2 pad 2: GND -> Net-(D2-Pad2)
- D3 pad 1: Net-(D3-Pad1) -> GND
- D3 pad 2: GND -> Net-(D3-Pad2)
- R11 pad 2: Net-(D1-Pad1) -> Net-(D1-Pad2)
- R12 pad 2: Net-(D2-Pad1) -> Net-(D2-Pad2)
- R13 pad 2: Net-(D3-Pad1) -> Net-(D3-Pad2)
Routing:
- net Net-(F1-Pad1): track 31.6 -> 35.1 mm
- net CANL: track 35.3 -> 38.7 mm, vias 0 -> 1
- net Net-(D2-Pad2): track 0.00 -> 1.68 mm
- net Net-(D2-Pad1): track 1.68 -> 0.00 mm
- net Net-(D1-Pad2): track 0.00 -> 1.68 mm
- net Net-(D1-Pad1): track 1.68 -> 0.00 mm
- net Net-(D3-Pad2): track 0.00 -> 1.68 mm
- net Net-(D3-Pad1): track 1.68 -> 0.00 mm
- net CANH: track 33.5 -> 34.5 mm
- net Net-(P2-Pad1): track 21.4 -> 22.3 mm
Other:
- board text added: "DIYPinball CAN Cape Version 1.1"
- board text removed: "DIYPinball CAN Cape Version 1.0"
