File: beaglebone-can-r1.sch (KiCad schematic (older format))
At the start: 38 parts, among them P1 BEAGLEBONE_BLACK, P2 PINBALL-CONNECTOR, P3 PINBALL-CONNECTOR, U1 MCP2562, U2 24C256, U3 AP3513E

Commit message: A bunch of old updates
Parts:
- C1, C10, C11, C2, C3, C4, C5: symbol C -> C-RESCUE-beaglebone-can-r1
- C6, C7, C8, C9: symbol CP -> CP-RESCUE-beaglebone-can-r1
- R1, R10, R11, R12, R13, R2, R3, R4, R5, R6, R7, R8, R9: symbol R -> R-RESCUE-beaglebone-can-r1
Connections:
- net GND: now also D1.1 (K), D2.1 (K), D3.1 (K); no longer D1.2 (A), D2.2 (A), D3.2 (A)
- net at R11.2: now also D1.2 (A); no longer D1.1 (K)
- net at R12.2: now also D2.2 (A); no longer D2.1 (K)
- net at R13.2: now also D3.2 (A); no longer D3.1 (K)
Changed lines of the file:
@@
 EESchema Schematic File Version 2
+LIBS:beaglebone-can-r1-rescue
 LIBS:power
 LIBS:device
@@
 LIBS:memory
 LIBS:xilinx
-LIBS:special
 LIBS:microcontrollers
 LIBS:dsp
@@
 $EndComp
 $Comp
-L GND #PWR01
+L GND-RESCUE-beaglebone-can-r1 #PWR01
 U 1 1 5458579E
 P 1400 4200
@@
 $EndComp
 $Comp
-L GND #PWR02
+L GND-RESCUE-beaglebone-can-r1 #PWR02
 U 1 1 545857B2
 P 2400 4200
@@
 $EndComp
 $Comp
-L GND #PWR03
+L GND-RESCUE-beaglebone-can-r1 #PWR03
 U 1 1 545857C6
 P 3400 4200
@@
 $EndComp
 $Comp
-L GND #PWR04
+L GND-RESCUE-beaglebone-can-r1 #PWR04
 U 1 1 545857DA
 P 4400 4200
@@
 Connection ~ 2400 4100
 $Comp
-L +3.3V #PWR05
+L +3.3V-RESCUE-beaglebone-can-r1 #PWR05
 U 1 1 54585853
 P 2500 1800
@@
 $EndComp
 $Comp
-L +3.3V #PWR06
+L +3.3V-RESCUE-beaglebone-can-r1 #PWR06
 U 1 1 54585867
 P 1300 1800
@@
 	2300 3100 2500 3100
 $Comp
-L R R4
+L R-RESCUE-beaglebone-can-r1 R4
 U 1 1 54585F9E
 P 9500 4350
@@
 $EndComp
 $Comp
-L R R5
+L R-RESCUE-beaglebone-can-r1 R5
 U 1 1 54586055
 P 9700 4350
@@
 $EndComp
 $Comp
-L R R3
+L R-RESCUE-beaglebone-can-r1 R3
 U 1 1 5458606E
 P 7700 4350
@@
 $EndComp
 $Comp
-L R R2
+L R-RESCUE-beaglebone-can-r1 R2
 U 1 1 54586087
 P 7500 4350
@@
 $EndComp
 $Comp
-L R R1
+L R-RESCUE-beaglebone-can-r1 R1
 U 1 1 545860A0
 P 7300 4350
@@
 Connection ~ 7500 4000
 $Comp
-L R R6
+L R-RESCUE-beaglebone-can-r1 R6
 U 1 1 54586641
 P 9900 5450
@@
 	8600 5400 8600 5900
 $Comp
-L GND #PWR09
+L GND-RESCUE-beaglebone-can-r1 #PWR09
 U 1 1 545867AA
 P 8600 5900
@@
 Connection ~ 8600 5800
 $Comp
-L +3.3V #PWR010
+L +3.3V-RESCUE-beaglebone-can-r1 #PWR010
 U 1 1 545868E3
 P 7300 3900
@@
 Connection ~ 9700 4000
 $Comp
-L C C3
+L C-RESCUE-beaglebone-can-r1 C3
 U 1 1 54587CAC
 P 7100 4900
@@
 $EndComp
 $Comp
-L GND #PWR011
+L GND-RESCUE-beaglebone-can-r1 #PWR011
 U 1 1 5458695B
 P 8000 2750
@@
 $EndComp
 $Comp
-L +3.3V #PWR013
+L +3.3V-RESCUE-beaglebone-can-r1 #PWR013
 U 1 1 54586983
 P 9200 2250
@@
 	9300 2450 9100 2450
 $Comp
-L C C2
+L C-RESCUE-beaglebone-can-r1 C2
 U 1 1 54586E51
 P 7200 2500
@@
 $EndComp
 $Comp
-L C C1
+L C-RESCUE-beaglebone-can-r1 C1
 U 1 1 545871EE
 P 6900 2500
@@
 $EndComp
 $Comp
-L GND #PWR014
+L GND-RESCUE-beaglebone-can-r1 #PWR014
 U 1 1 5458721A
 P 6900 2750
@@
 $EndComp
 $Comp
-L GND #PWR015
+L GND-RESCUE-beaglebone-can-r1 #PWR015
 U 1 1 54587235
 P 7200 2750
@@
 $EndComp
 $Comp
-L +3.3V #PWR017
+L +3.3V-RESCUE-beaglebone-can-r1 #PWR017
 U 1 1 5458738B
 P 7200 2250
@@
 Connection ~ 1600 5850
 $Comp
-L GND #PWR018
+L GND-RESCUE-beaglebone-can-r1 #PWR018
 U 1 1 5571C3FE
 P 1600 7900
@@
 $EndComp
 $Comp
-L GND #PWR020
+L GND-RESCUE-beaglebone-can-r1 #PWR020
 U 1 1 5571E52E
 P 7950 1700
@@
 Connection ~ 7950 1600
 $Comp
-L R R7
+L R-RESCUE-beaglebone-can-r1 R7
 U 1 1 5571E538
 P 7250 1000
@@
 $EndComp
 $Comp
-L C C11
+L C-RESCUE-beaglebone-can-r1 C11
 U 1 1 5571E53F
 P 6250 1600
@@
 $EndComp
 $Comp
-L R R8
+L R-RESCUE-beaglebone-can-r1 R8
 U 1 1 5571E546
 P 5700 1600
@@
 $EndComp
 $Comp
-L C C10
+L C-RESCUE-beaglebone-can-r1 C10
 U 1 1 5571E54D
 P 6000 1450
@@
 $EndComp
 $Comp
-L C C4
+L C-RESCUE-beaglebone-can-r1 C4
 U 1 1 5571E554
 P 6000 1200
@@
 	6050 1600 5950 1600
 $Comp
-L GND #PWR021
+L GND-RESCUE-beaglebone-can-r1 #PWR021
 U 1 1 5571E564
 P 5350 1900
@@
 Connection ~ 5350 1600
 $Comp
-L C C5
+L C-RESCUE-beaglebone-can-r1 C5
 U 1 1 5571E570
 P 8250 1200
@@
 Connection ~ 8550 1400
 $Comp
-L R R9
+L R-RESCUE-beaglebone-can-r1 R9
 U 1 1 5571E587
 P 5700 1800
@@
 $EndComp
 $Comp
-L R R10
+L R-RESCUE-beaglebone-can-r1 R10
 U 1 1 5571E58E
 P 6400 1800
@@
 Connection ~ 7950 1000
 $Comp
-L CP C8
+L CP-RESCUE-beaglebone-can-r1 C8
 U 1 1 5571E5B0
 P 4850 1400
@@
 $EndComp
 $Comp
-L CP C9
+L CP-RESCUE-beaglebone-can-r1 C9
 U 1 1 5571E5B7
 P 5150 1400
@@
 Connection ~ 5150 900
 $Comp
-L CP C6
+L CP-RESCUE-beaglebone-can-r1 C6
 U 1 1 5571E5C4
 P 9500 1300
@@
 $EndComp
 $Comp
-L CP C7
+L CP-RESCUE-beaglebone-can-r1 C7
 U 1 1 5571E5CB
 P 9750 1300
@@
 Connection ~ 9500 1000
 $Comp
-L GND #PWR024
+L GND-RESCUE-beaglebone-can-r1 #PWR024
 U 1 1 5571E5DA
 P 9500 1700
@@
 Connection ~ 9500 1600
 $Comp
-L R R11
+L R-RESCUE-beaglebone-can-r1 R11
 U 1 1 5571FFF6
 P 5350 6700
@@
 $EndComp
 $Comp
-L R R12
+L R-RESCUE-beaglebone-can-r1 R12
 U 1 1 5571FFFD
 P 5650 6700
@@
 $EndComp
 $Comp
-L R R13
+L R-RESCUE-beaglebone-can-r1 R13
 U 1 1 55720004
 P 5950 6700
@@
 $EndComp
 $Comp
-L LED D1
-U 1 1 5572000B
-P 5350 7350
-F 0 "D1" H 5350 7450 50  0000 C CNN
-F 1 "LED" H 5350 7250 50  0000 C CNN
-F 2 "LEDs:LED-0603" H 5350 7350 60  0001 C CNN
-F 3 "" H 5350 7350 60  0000 C CNN
-	1    5350 7350
-	0    1    1    0
-$EndComp
-$Comp
-L LED D2
-U 1 1 55720012
-P 5650 7350
-F 0 "D2" H 5650 7450 50  0000 C CNN
-F 1 "LED" H 5650 7250 50  0000 C CNN
-F 2 "LEDs:LED-0603" H 5650 7350 60  0001 C CNN
-F 3 "" H 5650 7350 60  0000 C CNN
-	1    5650 7350
-	0    1    1    0
-$EndComp
-$Comp
-L LED D3
-U 1 1 55720019
-P 5950 7350
-F 0 "D3" H 5950 7450 50  0000 C CNN
-F 1 "LED" H 5950 7250 50  0000 C CNN
-F 2 "LEDs:LED-0603" H 5950 7350 60  0001 C CNN
-F 3 "" H 5950 7350 60  0000 C CNN
-	1    5950 7350
-	0    1    1    0
-$EndComp
-$Comp
-L GND #PWR025
+L GND-RESCUE-beaglebone-can-r1 #PWR025
 U 1 1 55720020
 P 5650 7750
@@
 Wire Wire Line
 	1900 4950 1800 4950
+$Comp
+L LED D3
+U 1 1 5611DE25
+P 5950 7350
+F 0 "D3" H 5950 7450 50  0000 C CNN
+F 1 "LED" H 5950 7250 50  0000 C CNN
+F 2 "LEDs:LED-0603" H 5950 7350 60  0001 C CNN
+F 3 "" H 5950 7350 60  0000 C CNN
+	1    5950 7350
+	0    -1   -1   0
+$EndComp
+$Comp
+L LED D2
+U 1 1 5611DF81
+P 5650 7350
+F 0 "D2" H 5650 7450 50  0000 C CNN
+F 1 "LED" H 5650 7250 50  0000 C CNN
+F 2 "LEDs:LED-0603" H 5650 7350 60  0001 C CNN
+F 3 "" H 5650 7350 60  0000 C CNN
+	1    5650 7350
+	0    -1   -1   0
+$EndComp
+$Comp
+L LED D1
+U 1 1 5611E0AE
+P 5350 7350
+F 0 "D1" H 5350 7450 50  0000 C CNN
+F 1 "LED" H 5350 7250 50  0000 C CNN
+F 2 "LEDs:LED-0603" H 5350 7350 60  0001 C CNN
+F 3 "" H 5350 7350 60  0000 C CNN
+	1    5350 7350
+	0    -1   -1   0
+$EndComp
 $EndSCHEMATC
